File: schematics/led_blink/led_blink.kicad_sch (KiCad schematic)
At the start: 16 parts, among them J1 Conn_01x02_Male, Q1 Q_NPN_BCE, Q2 Q_NPN_BCE, Q3 Q_NPN_BCE, SW1 SW_Push, SW2 SW_Push, SW3 SW_Push, U1 TM4C123GH6PMI, Y1 Crystal

Commit message: dev
Other:
- company: (none) -> Sprints ARM master class
- title: (none) -> Led blink
Changed lines of the file:
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@@
 (kicad_sch (version 20211123) (generator eeschema)
   (paper "A4")
+  (title_block
+    (title "Led blink")
+    (date "2022-12-22")
+    (rev "Mohamed ABdelnasser")
+    (company "Sprints ARM master class")
+  )
   (junction (at 83.82 172.72) (diameter 0) (color 0 0 0 0)
   )
